File: pedals/DSPP-1/electrical/DSPP-1.kicad_sch (KiCad schematic)
At the start: 27 parts, among them J1 Guitar Jack, U1 STM32G474CBTx, U3 PCM3060, U4 OPA1678

Commit message: schematic update for MCU, Codec
Parts:
- removed C7: 2.2n, symbol Device:C_Small
- added C17, C28: 100n, Capacitor_SMD:C_0805_2012Metric, symbol Device:C_Small
- added C18: 10u, Capacitor_SMD:C_0805_2012Metric, symbol Device:C_Small
- added J2: USB_C, sumec_brd:USB_C_Receptacle_GCT_USB4105-xx-A_16P_TopMnt_Horizontal, symbol Connector:USB_C_Receptacle_USB2.0_16P
- added JP2, JP3: Jumper, Jumper:SolderJumper-3_P1.3mm_Open_RoundedPad1.0x1.5mm, symbol Jumper:SolderJumper_3_Open
- added Q1: SI2393DS, Package_TO_SOT_SMD:SOT-23-3, symbol Device:Q_PMOS_GSD
- added R12, R13, R15: 10k, Resistor_SMD:R_0805_2012Metric, symbol Device:R_Small
- added R14: 5.1k, Resistor_SMD:R_0805_2012Metric, symbol Device:R_Small
- added R21, R22: 15R, Resistor_SMD:R_0805_2012Metric, symbol Device:R_Small
- added U5: USBLC6-2SC6, Package_TO_SOT_SMD:SOT-23-6, symbol Power_Protection:USBLC6-2SC6
- added Y1, Y2: Crystal, symbol Device:Crystal
- C10, C11, C12, C13, C14, C15, C16, C2, C3, C4, C5, C6: footprint (none) -> Capacitor_SMD:C_0805_2012Metric
- J1: footprint (none) -> Connector_Audio:Jack_6.35mm_Neutrik_NMJ6HCD2_Horizontal
- JP1: footprint (none) -> Jumper:SolderJumper-3_P1.3mm_Open_RoundedPad1.0x1.5mm
- R10, R11, R3, R4, R5, R6, R7, R9: footprint (none) -> Resistor_SMD:R_0805_2012Metric
- R8: value 100R -> 5.1k; footprint (none) -> Resistor_SMD:R_0805_2012Metric
- U4: footprint (none) -> Package_SON:SON-8-1EP_3x2mm_P0.5mm_EP1.4x1.6mm
Connections:
- net BCK is gone; now on net SAI_SCK_A: U3.10 (BCK2), U3.5 (BCK1)
- net LRCK is gone; now on net SAI_FS_A: U3.11 (LRCK2), U3.4 (LRCK1)
- net SCKI is gone; now on net SAI_MCLK_A: U3.6 (SCKI1), U3.9 (SCKI2)
- net +3V3: now also R12.1, R13.1
- net AUDIO_CODEC_IN: no longer R8.1
- net GND: now also R8.1, U1.23 (VSS), U1.35 (VSS), U1.47 (VSS), C28.2, J2.A1 (GND), J2.A12 (GND), J2.B1 (GND), J2.B12 (GND), J2.S1 (SHIELD), R14.1, U5.2 (GND)
- net SCL: now also JP3.2 (C), R13.2
- net SDA: now also JP2.2 (C), R12.2
- net SAI_SD_A: now reaches U3.12 (DIN)
- net SAI_SD_A: now also U1.32 (PA10)
- net SAI_SD_B: now reaches U3.3 (DOUT)
- net SAI_SD_B: now also U1.42 (PB5)
- net at R8.2: now also J2.B5 (CC2)
- net at U1.1 (VBAT): now also U1.21 (VDDA), U1.24 (VDD), U1.36 (VDD), U1.48 (VDD)
- net SAI_MCLK_A: now reaches U1.11 (PA3)
- net SAI_SCK_A: now reaches U1.30 (PA8)
- net SAI_FS_A: now reaches U1.31 (PA9)
- net D-: now reaches U1.33 (PA11)
- net D-: now also U5.6 (I/O1)
- net D+: now reaches U1.34 (PA12)
- net D+: now also U5.4 (I/O2)
- net at U1.39 (PA15): now also JP3.1 (A)
- net at U1.44 (PB7): now also JP2.1 (A)
- new net: J2.A7 (D-), J2.B7 (D-), R22.1
- new net: J2.A6 (D+), J2.B6 (D+), R21.1
- new net: J2.A5 (CC1), R14.2
- new net DN_IN: R22.2, U5.1 (I/O1)
- new net DP_IN: R21.2, U5.3 (I/O2)
- new net MSW_ON: Q1.1 (G), R15.1
- new net USB_VBUS: C28.1, J2.A4 (VBUS), J2.A9 (VBUS), J2.B4 (VBUS), J2.B9 (VBUS), U5.5 (VBUS)
- new net VIN: Q1.3 (D)
- new net VSYS: Q1.2 (S), R15.2
- no-connect marks 0 -> 2
Other:
- note added: "1. 2. 3. 4. 5. 6. 7."
- note added: "Ferrite beads for analog"
- note added: "MAIN SW"
- note added: "MCU and CODEC"
- note added: "POWER MANAGEMENT"
- note added: "Rds On = 22.7 mOhms Vds = 30 V Vgs = - 20 V, + 16 V Vgs th = 2.2 V"
- note added: "TO-DO LIST"
- note added: "USB C CONNECTOR"
- note removed: "LPF"
- moved on the sheet: C10, C11, C12, C13, C14, C15, C16, C2, C3, C4, C5, C6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

Commit message: updated schematic added docs
Parts:
- added C19, C21, C23, C25, C30, C34: 100n, Capacitor_SMD:C_0805_2012Metric, symbol Device:C_Small
- added C20, C22, C24, C26: 10u, Capacitor_SMD:C_0805_2012Metric, symbol Device:C_Small
- added C31, C32, C33, C35, C36: 22u, Capacitor_SMD:C_0805_2012Metric, symbol Device:C_Small
- added D1: SD0805S020S0R5, Diode_SMD:D_0805_2012Metric, symbol Device:D_Schottky
- added FB1: 742792042, Inductor_SMD:L_0805_2012Metric, symbol Device:FerriteBead_Small
- added H1, H2, H3, H4: M3, symbol Mechanical:MountingHole_Pad
- added IC2: TPS565247DRLR, SOTFL50P160X60-6N, symbol SamacSys_Parts:TPS565247DRLR
- added IC3: TLV77333PDBVR, Package_TO_SOT_SMD:SOT-23-5, symbol SamacSys_Parts:TLV77333PDBVR
- added J3: BarrelJack, symbol Connector:Barrel_Jack_MountingPin
- added L2: 2.2u, Inductor_SMD:L_1008_2520Metric, symbol Device:L_Small
- added R19: 82k, Resistor_SMD:R_0805_2012Metric, symbol Device:R_Small
- added R20: 10k, Resistor_SMD:R_0805_2012Metric, symbol Device:R_Small
- added SW1: SW_Nidec_CAS-120A1, Button_Switch_SMD:Nidec_Copal_CAS-120A, symbol Switch:SW_Nidec_CAS-120A1
- added U2: TPS7A20xxxDBV, Package_TO_SOT_SMD:SOT-23-5, symbol Regulator_Linear:TPS7A20xxxDBV
Connections:
- net VSYS is gone; now on net VIN: Q1.2 (S), R15.2
- net +3V3: now also C23.2, C24.2, IC3.5 (OUT)
- net +5VA: now also C19.2, C20.2, U2.5 (OUT)
- net GND: now also C19.1, C20.1, C21.1, C22.1, C23.1, C24.1, C25.1, C26.1, C30.2, C31.2, C32.2, C33.2, C34.2, C35.2, C36.2, H1.1, H2.1, H3.1, H4.1, IC2.3 (GND), IC2.4 (AGND), IC3.2 (GND), J3.1, J3.MP (MountPin), R20.1, SW1.2 (B), U2.2 (GND); no longer U3.16 (SGND), U3.22 (AGND2), U3.23 (AGND1), U3.8 (DGND)
- net VIN: now also D1.1 (K); no longer Q1.3 (D)
- net MSW_ON: no longer names the net of Q1.1 (G), R15.1
- net MSW_ON: now also SW1.3 (A)
- new net: D1.2 (A), J3.2
- new net: C21.2, C22.2, FB1.2, U2.1 (IN), U2.3 (EN)
- new net: IC2.6 (FB), R19.1, R20.2
- new net: IC2.2 (SW), L2.1
- new net +5V5: C25.2, C26.2, C30.1, C31.1, C32.1, C33.1, FB1.1, IC3.1 (IN), IC3.3 (EN), L2.2, R19.2
- new net VCC: C34.1, C35.1, C36.1, IC2.1 (VIN), IC2.5 (EN), Q1.3 (D)
- no-connect marks 2 -> 3
Other:
- note added: "1. Footswitch, pots (UI PART) 2. 3. 4. 5. 6. 7."
- note added: "ANALOG CIRCUIT"
- note added: "ANALOG LDO"
- note added: "BR. JACK"
- note added: "Center neagtive (like most guitar pedals)"
- note added: "Current draw: STM32G4 - 25mA OpAmps - 5mA Codec - 21mA"
- note added: "DIGITAL LDO"
- note added: "MOUNT. and TPs"
- note added: "MOUNTING"
- note added: "OFF"
- note added: "ON"
- note added: "POWER MANAGEMENT and SOURCES"
- note added: "STEP-DOWN CONVERTER 5.5V"
- note added: "TPs"
- note removed: "1. 2. 3. 4. 5. 6. 7."
- note removed: "POWER MANAGEMENT"
- note removed: "Rds On = 22.7 mOhms Vds = 30 V Vgs = - 20 V, + 16 V Vgs th = 2.2 V"
- moved on the sheet: C10, C11, C12, C13, C14, C15, C16, C17, C18, C2, C28, C3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

Commit message: Updated schematic, STM32 pinout
Parts:
- removed JP2, JP3: Jumper, Jumper:SolderJumper-3_P1.3mm_Open_RoundedPad1.0x1.5mm, symbol Jumper:SolderJumper_3_Open
- removed R12: 10k, Resistor_SMD:R_0805_2012Metric, symbol Device:R_Small
- removed Y1: Crystal, symbol Device:Crystal
- added C31, C32: 30p, Capacitor_SMD:C_0603_1608Metric, symbol Device:C_Small
- added C33: 10u, Capacitor_SMD:C_0805_2012Metric, symbol Device:C_Small
- added C34, C35, C36, C37: 100n, Capacitor_SMD:C_0805_2012Metric, symbol Device:C_Small
- added FB2: 742792042, Inductor_SMD:L_0805_2012Metric, symbol Device:FerriteBead_Small
- added R10: 10k, Resistor_SMD:R_0805_2012Metric, symbol Device:R_Small
- added R4, R5: 100k, Resistor_SMD:R_0805_2012Metric, symbol Device:R_Small
- R2: renamed from R19; value 82k -> 76.8k
- SW1: value SW_Nidec_CAS-120A1 -> SW; footprint Button_Switch_SMD:Nidec_Copal_CAS-120A -> (none)
- U1: renamed from U2; value TPS7A20xxxDBV -> TPS7A2055PDBVRG4
- U3: renamed from U1; value STM32G474CBTx -> STM32G474CBT6TR
- Y2: value Crystal -> ABLS-12.288; footprint (none) -> Crystal:Crystal_SMD_HC49-SD
- renumbered C22 to C1, C23 to C10, C30 to C11, C24 to C12, C31 to C13, C32 to C14, C33 to C15, C28 to C16, C18 to C17, C17 to C18, C5 to C19, C21 to C2, C6 to C20, C2 to C21, C3 to C22, C4 to C23, C16 to C24, C11 to C25, C10 to C26, C13 to C27, C12 to C28, C14 to C29, C19 to C3, C15 to C30, C20 to C4, C26 to C5, C25 to C6, C34 to C7, C35 to C8, C36 to C9, IC3 to IC1, J3 to J1, J1 to J3, L2 to L1, R15 to R1, R13 to R11, R7 to R12, R5 to R13, R6 to R14, R3 to R15, R4 to R16, R9 to R17, R11 to R18, R10 to R19, R20 to R3, R8 to R6, R22 to R7, R21 to R8, R14 to R9, U5 to U2, U3 to U5
Connections:
- net +3V3: now also U3.1 (VBAT), U3.24 (VDD), U3.36 (VDD), U3.48 (VDD), C33.2, C34.2, C35.2, C36.2, C37.2, FB2.1, R10.1
- net GND: now also C17.1, C18.1, C31.2, C32.2, C33.1, C34.1, C35.1, C36.1, C37.1, R5.1
- net SAI_SCK_A: now also U3.22 (PB10); no longer U3.30 (PA8)
- net SCL: now also U3.39 (PA15)
- net SDA: now also U3.44 (PB7), R10.2
- net VCC: now also R4.2; no longer IC2.5 (EN)
- net VDDA: now reaches C17.2
- net VDDA: now also C18.2, U3.20 (VREF+), U3.21 (VDDA), FB2.2
- net at Y2.1: now also U3.5 (PF0), C32.1
- net at Y2.2: now also U3.6 (PF1), C31.1
- net SWDIO: now reaches U3.37 (PA13)
- net SWCLK: now reaches U3.38 (PA14)
- net SWO: now reaches U3.40 (PB3)
- net BOOT0: now reaches U3.45 (PB8)
- net NRST: now reaches U3.7 (PG10)
- net +5V5 renamed +5V2
- new net: IC2.5 (EN), R4.1, R5.2
Other:
- note added: "1. Footswitch, pots (UI PART) 2. Decide what kind of grounding to use 3. 4. 5. 6. 7."
- note removed: "1. Footswitch, pots (UI PART) 2. 3. 4. 5. 6. 7."
- moved on the sheet: C1, C10, C11, C12, C13, C14, C15, C16, C17, C18, C2, C24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
