File: pedals/DSPP-1/electrical/DSPP-1.kicad_sch (KiCad schematic)
At the start: 78 parts, among them IC1 TLV77333PDBVR, IC2 TPS565247DRLR, J1 BarrelJack, J2 USB_C, J3 Guitar Jack, Q1 SI2393DS, SW1 SW, U1 TPS7A2055PDBVRG4, U2 USBLC6-2SC6, U3 STM32G474CBT6TR, U4 OPA1678, U5 PCM3060, Y2 ABLS-12.288

Commit message: updates schematic added LEDs, memory, storage
Parts:
- removed R10: 10k, Resistor_SMD:R_0805_2012Metric, symbol Device:R_Small
- added C12, C2, C27, C28: 10u, Capacitor_SMD:C_0805_2012Metric, symbol Device:C_Small
- added C19, C30, C31, C37: 100n, Capacitor_SMD:C_0805_2012Metric, symbol Device:C_Small
- added D2: LED, symbol Device:LED_Small
- added D3, D4, D5: LED, LED_SMD:LED_0805_2012Metric, symbol Device:LED
- added J3: SWD, Connector_PinHeader_1.27mm:PinHeader_2x05_P1.27mm_Vertical_SMD, symbol Connector_Generic:Conn_02x05_Odd_Even
- added J4: DM3AT, Connector_Card:microSD_HC_Hirose_DM3AT-SF-PEJM5, symbol Connector:Micro_SD_Card_Det2
- added JP1: Jumper_2_Small_Open, Jumper:SolderJumper-2_P1.3mm_Open_RoundedPad1.0x1.5mm, symbol Jumper:Jumper_2_Small_Open
- added R1, R25, R26, R27, R28, R31, R32, R37, R38: 10k, Resistor_SMD:R_0805_2012Metric, symbol Device:R_Small
- added R12, R13, R14, R15, R2, R3, R30, R4, R5, R6: 22R, Resistor_SMD:R_0805_2012Metric, symbol Device:R_Small
- added R29: 2.2k, Resistor_SMD:R_0805_2012Metric, symbol Device:R_Small
- added R39: 0/220k, Resistor_SMD:R_0805_2012Metric, symbol Device:R_Small
- added R40, R41, R42: 2.2k, Resistor_SMD:R_0805_2012Metric, symbol Device:R
- added SW2: Button, symbol Switch:SW_MEC_5G
- added SW3: SW, symbol Switch:SW_Nidec_CAS-120A1
- added SW4: RESET, symbol Switch:SW_MEC_5G
- added TP1, TP2, TP3, TP4, TP5, TP6, TP7, TP8: TestPoint, TestPoint:TestPoint_Pad_D1.0mm, symbol Connector:TestPoint
- added U1, U3: LM66100DCKR, Package_TO_SOT_SMD:SOT-363_SC-70-6, symbol Power_Management:LM66100DCK
- added U6: APS6404L-3SQRx-SN, Package_SO:SOIC-8_3.9x4.9mm_P1.27mm, symbol Memory_RAM:APS6404L-3SQRx-SN
- added U7: 24CW1280T-I/OT, Package_TO_SOT_SMD:SOT-23-5, symbol Memory_EEPROM:24AA02-OT
- R11: value 10k -> 22R
- R18: value 0/220k -> 10k
- renumbered C33 to C1, C37 to C10, C21 to C11, C18 to C13, C17 to C14, C1 to C15, C22 to C16, C23 to C17, C2 to C18, C3 to C20, C4 to C21, C7 to C22, C5 to C23, C8 to C24, C6 to C25, C9 to C26, C11 to C29, C34 to C3, C13 to C32, C14 to C33, C10 to C34, C15 to C35, C12 to C36, C16 to C38, C24 to C39, C32 to C4, C25 to C40, C26 to C41, C27 to C42, C28 to C43, C29 to C44, C30 to C45, C31 to C5, C35 to C6, C19 to C7, C36 to C8, C20 to C9, FB2 to FB1, FB1 to FB2, IC2 to IC1, IC1 to IC2, J3 to J1, J1 to J2, J2 to J5, JP1 to JP2, R1 to R10, R15 to R16, R16 to R17, R17 to R19, R19 to R20, R2 to R21, R3 to R22, R4 to R23, R5 to R24, R6 to R33, R7 to R34, R8 to R35, R9 to R36, R12 to R7, R13 to R8, R14 to R9, U4 to U2, U3 to U4, U1 to U5, U2 to U8, U5 to U9, Y2 to Y1
Connections:
- net +3V3: now also R18.1, C27.2, C28.2, C30.2, C31.2, C37.2, J3.1 (Pin_1), J4.4 (VDD), JP1.2 (B), R1.1, R26.2, R27.1, R29.1, R31.2, R32.2, R38.2, R42.1, SW3.3 (A), U6.8 (VDD), U7.4 (V_{CC}); no longer R11.1
- net +5V2: now also C2.2, U1.1 (VIN), U3.3 (~{CE}); no longer C23.2, C25.2, FB2.1, IC2.1 (IN), IC2.3 (EN)
- net +5VA: now also R41.1
- net BOOT0: now also R25.1
- net GND: now also U4.19 (VSSA), U9.22 (AGND2), U9.23 (AGND1), U9.8 (DGND), C12.1, C19.1, C2.1, C27.1, C28.1, C30.1, C31.1, C37.1, D3.1 (K), D4.1 (K), D5.1 (K), J3.3 (Pin_3), J3.5 (Pin_5), J3.9 (Pin_9), J4.6 (VSS), J4.9 (DET_B), J4.SH (SHIELD), R28.2, R37.1, SW2.3 (B), SW2.4 (B), SW3.1 (C), SW4.3 (B), SW4.4 (B), U1.2 (GND), U3.2 (GND), U6.4 (VSS), U7.2 (V_{SS})
- net NRST: now also C19.2, J3.10 (Pin_10), R26.1, SW2.1 (A), SW2.2 (A)
- net SAI_FS_A: now also R15.2; no longer U4.31 (PA9)
- net SAI_MCLK_A: now also R11.2; no longer U4.11 (PA3)
- net SAI_SCK_A: now also R14.2; no longer U4.22 (PB10)
- net SCL: now also R18.2, U7.1 (SCL); no longer R11.2
- net SDA: now also R1.2, U7.3 (SDA)
- net SWCLK: now also J3.4 (Pin_4), R28.1
- net SWDIO: now also J3.2 (Pin_2), R27.2
- net SWO: now also J3.6 (Pin_6)
- net USB_VBUS: now also C12.2, R40.1, TP5.1, U1.3 (~{CE}), U3.1 (VIN)
- net VCC: now also C23.2, C25.2, FB2.1, IC2.1 (IN), IC2.3 (EN), U1.6 (VOUT), U3.6 (VOUT); no longer C22.1, C24.1, C26.1, IC1.1 (VIN), Q1.3 (D), R23.2
- net at U9.28 (MODE): now also R39.2; no longer R18.2
- net at JP2.2 (C): now also R39.1; no longer R18.1
- net QSPI_CS: now reaches U4.10 (PA2)
- net QSPI_CS: now also R32.1, U6.1 (~{CE})
- net at U4.14 (PA6): now also R12.1
- net at U4.15 (PA7): now also R13.1
- net at U4.16 (PB0): now also R2.2
- net at U4.17 (PB1): now also R3.2
- net at U4.27 (PB13): now also R5.2
- net SPI_MISO: now reaches U4.28 (PB14)
- net SPI_MISO: now also R30.1
- net at U4.29 (PB15): now also R6.2
- net at U4.30 (PA8): now also R14.1
- net ADRR: no longer names the net of U9.27 (~{MS}/AD/IFMD)
- net ADRR: now also JP1.1 (A), R37.2
- net ~{RST}: no longer names the net of U9.15 (~{RST})
- net ~{RST}: now also R38.1, SW4.1 (A), SW4.2 (A)
- new net: R25.2, SW3.2 (B)
- new net: D4.2 (A), R41.2
- new net: D2.2 (A), R29.2
- new net: D3.2 (A), R40.2
- new net: D5.2 (A), R42.2
- new net: D2.1 (K), J4.10 (DET_A)
- new net: J4.7 (DAT0), R30.2
- new net: R11.1, U4.11 (PA3)
- new net: R15.1, U4.31 (PA9)
- new net: R4.2, U4.22 (PB10)
- new net DSEL: TP8.1
- new net IO41: TP4.1
- new net IO42: TP2.1
- new net IO48: TP6.1
- new net QSPI_CLK: R4.1, U6.6 (SCLK)
- new net QSPI_IO0: R3.1, U6.5 (SI/SIO0)
- new net QSPI_IO1: R2.1, U6.2 (SO/SIO1)
- new net QSPI_IO2: R13.2, U6.3 (SIO2)
- new net QSPI_IO3: R12.2, U6.7 (SIO3)
- new net SPI_CLK: J4.5 (CLK), R5.1
- new net SPI_CS: J4.2 (DAT3/CD), R31.1
- new net SPI_MOSI: J4.3 (CMD), R6.1
- new net VBATT: TP3.1
- new net VOTG: TP7.1
- new net VSYS: C22.1, C24.1, C26.1, IC1.1 (VIN), Q1.3 (D), R23.2, TP1.1
- no-connect marks 3 -> 10
Other:
- note added: "1. Footswitch, pots (UI PART) 2. Decide what kind of grounding to use 3. SD card 4. Memory for looping 5. 6. 7."
- note added: "BOOT SLCT"
- note added: "DEBUG"
- note added: "DSPP-1"
- note added: "EEPROM"
- note added: "I2C Addr.: 0x50"
- note added: "LEDs"
- note added: "MCU and PERIHPERALS"
- note added: "MEMORY and STORAGE"
- note added: "NORMAL"
- note added: "OUTPUT BUFFER STAGE"
- note added: "POWER OR-ING"
- note added: "QSPI PSRAM"
- note added: "RESET"
- note added: "SC CARD"
- note added: "SWD CONN"
- note added: "SWITCHES, POTS, LEDs"
- note added: "TEST POINTS"
- note added: "pinout checked"
- note removed: "1. Footswitch, pots (UI PART) 2. Decide what kind of grounding to use 3. 4. 5. 6. 7."
- note removed: "Ferrite beads for analog"
- note removed: "MCU and CODEC"
- note removed: "TPs"
- company: bismarx -> bismarx-v1
- title: looper-v1 -> DSPP-1
- moved on the sheet: C1, C10, C11, C13, C14, C15, C16, C17, C18, C20, C21, C22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
