File: pedals/DSPP-1/electrical/DSPP-1.kicad_sch (KiCad schematic)
At the start: 131 parts, among them IC1 TPS565247DRLR, IC2 TLV77333PDBVR, J1 Guitar Jack, J2 BarrelJack, J3 SWD, J4 DM3AT, J5 USB_C, Q1 SI2393DS, SW1 SW, SW2 Button, SW3 SW, SW4 RESET, U1 LM66100DCKR, U2 OPA1678, U3 LM66100DCKR, U4 STM32G474CBT6TR, U5 TPS7A2055PDBVRG4, U6 APS6404L-3SQRx-SN, U7 24CW1280T-I/OT, U8 USBLC6-2SC6, U9 PCM3060, Y1 ABLS-12.288

Commit message: new 3d models, schematic update
Parts:
- removed D1: SD0805S020S0R5, Diode_SMD:D_0805_2012Metric, symbol Device:D_Schottky
- added D1: LED, symbol Device:LED_Small
- added D2: SD0805S020S0R5, Diode_SMD:D_0805_2012Metric, symbol Device:D_Schottky
- added D3: LED, LED_THT:LED_D2.0mm_W4.8mm_H2.5mm_FlatTop, symbol Device:LED_Small
- added J6: Guitar Jack, Connector_Audio:Jack_6.35mm_Neutrik_NMJ6HCD2_Horizontal, symbol Connector_Audio:AudioJack3_Ground_Switch
- added J7: OLED, inset_footprint:OLED DISPLAY, symbol Connector_Generic:Conn_01x04
- added R30: 10k, Resistor_SMD:R_0805_2012Metric, symbol Device:R_Small
- added R31, R8: 2.2k, Resistor_SMD:R_0805_2012Metric, symbol Device:R_Small
- added RV1: 100k, symbol Device:R_Potentiometer
- added SW1: SW_3PDT, SamacSys_Parts:STOMP-SWITCH-3PDT, symbol SamacSys_Parts:SW_Push_3PDT
- added SW5: FOOTSW_3PDT, SamacSys_Parts:STOMP-SWITCH-3PDT, symbol SamacSys_Parts:SW_Push_3PDT
- added U10: OPA1678, symbol Amplifier_Operational:OPA1678
- SW2: renamed from SW1; value SW -> SW_SPDT
- renumbered C9 to C11, C16 to C15, C17 to C16, C15 to C17, C30 to C29, C31 to C30, C29 to C31, C11 to C9, D2 to D4, D3 to D5, D4 to D6, D5 to D7, R9 to R10, R16 to R11, R17 to R12, R10 to R13, R11 to R14, R12 to R15, R13 to R16, R14 to R17, R15 to R18, R18 to R20, R20 to R21, R21 to R22, R22 to R23, R23 to R24, R24 to R25, R25 to R26, R26 to R27, R27 to R28, R28 to R29, R29 to R32, R30 to R33, R31 to R34, R32 to R35, R33 to R36, R34 to R37, R35 to R38, R36 to R39, R37 to R40, R38 to R41, R39 to R42, R40 to R43, R41 to R44, R42 to R45, R8 to R9, SW2 to SW3, SW3 to SW4, SW4 to SW6
Connections:
- net +3V3: now also R30.2, R31.1, R8.1
- net AUDIO_CODEC_IN: no longer R21.2
- net GND: now also J6.G, J6.S, SW1.1 (A), SW1.6 (C), SW1.8 (B), SW5.6 (C), SW5.9 (C); no longer J2.1
- net SCL: now also J7.3 (Pin_3)
- net SDA: now also J7.4 (Pin_4)
- net SPI_CS: now also U4.26 (PB12)
- net VCC: now also Q1.3 (D); no longer U1.6 (VOUT), U3.6 (VOUT)
- net VIN: now also C22.1, C24.1, C26.1, IC1.1 (VIN), R24.2, D2.1 (K); no longer Q1.2 (S), R13.2
- net VSYS: now also Q1.2 (S), R13.2, U1.6 (VOUT), U3.6 (VOUT); no longer C22.1, C24.1, C26.1, IC1.1 (VIN), Q1.3 (D), R24.2
- net CODEC_OUTPUT: now reaches U9.20 (V_{OUT}L+)
- net at J2.2: now also SW1.2 (B)
- net GNDBATT: now reaches J1.R
- new net: J2.1, SW1.5 (B)
- new net: D2.2 (A), SW1.3 (C), SW1.4 (A)
- new net: D1.1 (K), SW1.9 (C)
- new net: D1.2 (A), R8.2
- new net: D3.2 (A), R31.2
- new net: D3.1 (K), SW5.8 (B)
- new net BUFFERED_AUDIO: R21.2
- new net BUFFERED_BYPASS: SW5.1 (A)
- new net FOOTSW_IO: R30.1, SW5.5 (B)
- new net OUTPUT_AUDIO: J6.T, SW5.2 (B)
- new net PROCESSED_AUDIO: SW5.3 (C)
- no-connect marks 10 -> 16
Other:
- note added: "1. Footswitch, pots (UI PART) 2. Decide what kind of grounding to use 3. Check STM pinout 4. Do I need a displaY 5. 6. 7."
- note added: "BOX: https://www.tme.eu/cz/details/hm-1590bbk/univerzalni-krabicky/hammond/1590bbk/"
- note added: "CENTRE NEG"
- note added: "CENTRE NEG INDICATOR"
- note added: "CENTRE POS"
- note added: "Centre negative is used for most pedals"
- note added: "FOOTSWITCH, POTS, LEDS"
- note added: "FX ON INDICATOR"
- note removed: "1. Footswitch, pots (UI PART) 2. Decide what kind of grounding to use 3. SD card 4. Memory for looping 5. 6. 7."
- note removed: "Center neagtive (like most guitar pedals)"
- note removed: "SWITCHES, POTS, LEDs"
- moved on the sheet: C11, C15, C16, C22, C24, C26, C31, C32, C33, C35, C7, C9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
